Commit message: Added parameter to set truck and wheels

File: ros_arvi_description/urdf/arvi.urdf.xacro (robot description, xacro)
@@ -12,4 +12,12 @@
   <property name="M_PI" value="3.14159"/>
   <!-- Global properties -->
+  <!-- Wheels params -->
+  <property name="wheel_radius" value="0.035"/>
+  <property name="wheel_leght" value="0.03"/>
+  <property name="wheel_offset" value="0.023"/>
+  <property name="truck_offset_x" value="0.163"/>
+  <property name="truck_offset_y" value="0.0827"/>
+  <property name="truck_offset_z" value="0.024"/>
+  <!-- Wheels params -->
   <!-- base_link -->
   <link name="base_link">
@@ -210,6 +218,10 @@
   <!-- Plate -->
   <!-- Trucks -->
-  <xacro:left_truck parent="base_link"/>
-  <xacro:right_truck parent="base_link"/>
+  <xacro:left_truck parent="base_link" reflect="-1" wheel_off="${wheel_offset}">
+    <origin xyz="${truck_offset_x} ${truck_offset_y} ${truck_offset_z}" rpy="${M_PI/2} 0 ${M_PI}" />
+  </xacro:left_truck>
+  <xacro:right_truck parent="base_link" reflect="1" wheel_off="${-wheel_offset}">
+    <origin xyz="${truck_offset_x} ${-truck_offset_y} ${truck_offset_z}" rpy="${M_PI/2} 0 ${M_PI}" />
+  </xacro:right_truck>
   <!-- Trucks -->
 </robot>

File: ros_arvi_description/urdf/left_truck.urdf.xacro (robot description, xacro)
@@ -2,6 +2,5 @@
 <robot xmlns:xacro="http://ros.org/wiki/xacro" name="left_truck">
   <xacro:property name="path_left_truck" value="package://ros_arvi_description/meshes/left_truck" />
-  <xacro:property name="radius_wheel" value="0.035" />
-  <xacro:macro name="left_truck" params="parent">
+  <xacro:macro name="left_truck" params="parent reflect wheel_off *joint_pose">
   <link
     name="left_truck_Link">
@@ -33,5 +32,5 @@
 <xacro:if value="$(arg truck_fixed)">
   <joint name="left_truck" type="fixed">
-    <origin xyz="0.163050888156922 0.0827 0.02425" rpy="1.5707963267949 0 3.14159265358979" />
+    <xacro:insert_block name="joint_pose"/>
     <parent link="base_link" />
     <child link="left_truck_Link" />
@@ -41,5 +40,5 @@
 <xacro:unless value="$(arg truck_fixed)">
   <joint name="left_truck" type="revolute">
-    <origin xyz="0.163050888156922 0.0827 0.02425" rpy="1.5707963267949 0 3.14159265358979" />
+    <xacro:insert_block name="joint_pose"/>
     <parent link="base_link" />
     <child link="left_truck_Link" />
@@ -53,5 +52,5 @@
         <origin xyz="0 0 0" rpy="0 ${M_PI/2} 0" />
         <geometry>
-          <cylinder length="0.03" radius="${radius_wheel}"/>
+          <cylinder length="${wheel_leght}" radius="${wheel_radius}"/>
         </geometry>
         <material name="Black" />
@@ -60,5 +59,5 @@
         <origin xyz="0 0 0" rpy="0 ${M_PI/2} 0" />
         <geometry>
-            <cylinder length="0.03" radius="${radius_wheel}"/>
+          <cylinder length="${wheel_leght}" radius="${wheel_radius}"/>
         </geometry>
       </collision>
@@ -76,8 +75,8 @@
     </link>
     <joint name="left_active_sprocket" type="continuous">
-      <origin xyz="0.163050888156922 0.00999999999999986 ${0.00674999999999998+0.015}" rpy="0 1.5707963267949 0" />
+      <origin xyz="0.163050888156922 0.00999999999999986 ${wheel_off}" rpy="0 ${M_PI/2} 0" />
       <parent link="left_truck_Link" />
       <child link="left_active_sprocket_Link" />
-      <axis xyz="-1 0 0" />
+      <axis xyz="${reflect} 0 0" />
     </joint>
     <gazebo reference="left_active_sprocket_Link">
@@ -90,5 +89,5 @@
   <link name="left_passive_sprocket_Link">
     <inertial>
-      <origin xyz="-0.017586991668159 -1.20643425804978E-11 4.12712086728106E-11" rpy="0 0 0" />
+      <origin xyz="-0.017586991668159 0 0" rpy="0 0 0" />
       <mass value="0.0194093359138542" />
       <inertia
@@ -103,5 +102,5 @@
         <origin xyz="0 0 0" rpy="0 ${M_PI/2} 0" />
         <geometry>
-          <cylinder length="0.03" radius="${radius_wheel}"/>
+          <cylinder length="${wheel_leght}" radius="${wheel_radius}"/>
         </geometry>
         <material name="Black" />
@@ -110,13 +109,13 @@
         <origin xyz="0 0 0" rpy="0 ${M_PI/2} 0" />
         <geometry>
-            <cylinder length="0.03" radius="${radius_wheel}"/>
+            <cylinder length="${wheel_leght}" radius="${wheel_radius}"/>
         </geometry>
       </collision>
   </link>
   <joint name="left_passive_sprocket" type="continuous">
-    <origin xyz="-0.0450508881569225 0.00999999999999997 ${0.00550399999999998+0.015}" rpy="0 1.5707963267949 0" />
+    <origin xyz="-0.0450508881569225 0.00999999999999997 ${wheel_off}" rpy="0 ${M_PI/2} 0" />
     <parent link="left_truck_Link" />
     <child link="left_passive_sprocket_Link" />
-    <axis xyz="-1 0 0" />
+    <axis xyz="${reflect} 0 0" />
     <mimic joint="left_active_sprocket" multiplier="1" offset="0"/>
   </joint>
@@ -140,12 +139,12 @@
   </link>
   <joint name="left_active_sprocket" type="continuous">
-    <origin xyz="0.163050888156922 0.00999999999999986 0.00674999999999998" rpy="0 1.5707963267949 0" />
+    <origin xyz="0.163050888156922 0.00999999999999986 0.00674999999999998" rpy="0 ${M_PI/2} 0" />
     <parent link="left_truck_Link" />
     <child link="left_active_sprocket_Link" />
-    <axis xyz="-1 0 0" />
+    <axis xyz="${reflect} 0 0" />
   </joint>
   <link name="left_passive_sprocket_Link">
     <inertial>
-      <origin xyz="-0.017586991668159 -1.20643425804978E-11 4.12712086728106E-11" rpy="0 0 0" />
+      <origin xyz="-0.017586991668159 0 0" rpy="0 0 0" />
       <mass value="0.0194093359138542" />
       <inertia
@@ -175,5 +174,5 @@
     <parent link="left_truck_Link" />
     <child link="left_passive_sprocket_Link" />
-    <axis xyz="-1 0 0" />
+    <axis xyz="${reflect} 0 0" />
     <mimic joint="left_active_sprocket" multiplier="1" offset="0"/>
   </joint>

File: ros_arvi_description/urdf/right_truck.urdf.xacro (robot description, xacro)
@@ -2,6 +2,5 @@
 <robot xmlns:xacro="http://ros.org/wiki/xacro" name="right_truck">
   <xacro:property name="path_right_truck" value="package://ros_arvi_description/meshes/right_truck" />
-  <xacro:property name="radius_wheel" value="0.035" />
-  <xacro:macro name="right_truck" params="parent">
+  <xacro:macro name="right_truck" params="parent reflect wheel_off *joint_pose">
   <link name="right_truck_Link">
     <inertial>
@@ -32,5 +31,5 @@
 <xacro:if value="$(arg truck_fixed)">
   <joint name="right_truck" type="fixed">
-    <origin xyz="0.164050888156922 -0.0827 0.02425" rpy="1.5707963267949 8.1774002564028E-18 3.14159265358979" />
+    <xacro:insert_block name="joint_pose"/>
     <parent link="base_link" />
     <child link="right_truck_Link" />
@@ -40,5 +39,5 @@
 <xacro:unless value="$(arg truck_fixed)">
   <joint name="right_truck" type="revolute">
-    <origin xyz="0.164050888156922 -0.0827 0.02425" rpy="1.5707963267949 8.1774002564028E-18 3.14159265358979" />
+    <xacro:insert_block name="joint_pose"/>
     <parent link="base_link" />
     <child link="right_truck_Link" />
@@ -63,20 +62,20 @@
       <origin xyz="0 0 0" rpy="0 ${M_PI/2} 0" />
         <geometry>
-            <cylinder length="0.03" radius="${radius_wheel}"/>
-        </geometry>
-      <material name="Black" />
-    </visual>
-    <collision>
-      <origin xyz="0 0 0" rpy="0 ${M_PI/2} 0" />
-        <geometry>
-            <cylinder length="0.03" radius="${radius_wheel}"/>
+            <cylinder length="${wheel_leght}" radius="${wheel_radius}"/>
+        </geometry>
+      <material name="Black" />
+    </visual>
+    <collision>
+      <origin xyz="0 0 0" rpy="0 ${M_PI/2} 0" />
+        <geometry>
+            <cylinder length="${wheel_leght}" radius="${wheel_radius}"/>
         </geometry>
     </collision>
   </link>
   <joint name="right_active_sprocket" type="continuous">
-    <origin xyz="0.164050888156922 0.0100000000000001 ${-0.00674999999999994-0.015}" rpy="3.14159265358979 -1.5707963267949 0" />
+    <origin xyz="0.164050888156922 0.01 ${wheel_off}" rpy="${M_PI} ${-M_PI/2} 0" />
     <parent link="right_truck_Link" />
     <child link="right_active_sprocket_Link" />
-    <axis xyz="-1 0 0" />
+    <axis xyz="${reflect} 0 0" />
   </joint>
     <gazebo reference="right_active_sprocket_Link">
@@ -89,5 +88,5 @@
   <link name="right_passive_sprocket_Link">
     <inertial>
-      <origin xyz="-0.0175869916443205 -1.38659330545243E-10 1.11022302462516E-16" rpy="0 0 0" />
+      <origin xyz="-0.0175869916443205 0 0" rpy="0 0 0" />
       <mass value="0.0194093358554489" />
       <inertia
@@ -102,20 +101,20 @@
       <origin xyz="0 0 0" rpy="0 ${M_PI/2} 0" />
         <geometry>
-            <cylinder length="0.03" radius="${radius_wheel}"/>
-        </geometry>
-      <material name="Black" />
-    </visual>
-    <collision>
-      <origin xyz="0 0 0" rpy="0 ${M_PI/2} 0" />
-        <geometry>
-            <cylinder length="0.03" radius="${radius_wheel}"/>
+            <cylinder length="${wheel_leght}" radius="${wheel_radius}"/>
+        </geometry>
+      <material name="Black" />
+    </visual>
+    <collision>
+      <origin xyz="0 0 0" rpy="0 ${M_PI/2} 0" />
+        <geometry>
+            <cylinder length="${wheel_leght}" radius="${wheel_radius}"/>
         </geometry>
     </collision>
   </link>
   <joint name="right_passive_sprocket" type="continuous">
-    <origin xyz="-0.0440508881569224 0.01 ${-0.00550399999999997-0.015}" rpy="3.14159265358979 -1.5707963267949 0" />
+    <origin xyz="-0.0440508881569224 0.01 ${wheel_off}" rpy="${M_PI} ${-M_PI/2} 0" />
     <parent link="right_truck_Link" />
     <child link="right_passive_sprocket_Link" />
-    <axis xyz="-1 0 0" />
+    <axis xyz="${reflect} 0 0" />
     <mimic joint="right_active_sprocket" multiplier="1" offset="0"/>
   </joint>
@@ -159,9 +158,9 @@
     <parent link="right_truck_Link" />
     <child link="right_active_sprocket_Link" />
-    <axis xyz="-1 0 0" />
+    <axis xyz="${reflect} 0 0" />
   </joint>
   <link name="right_passive_sprocket_Link">
     <inertial>
-      <origin xyz="-0.0175869916443205 -1.38659330545243E-10 1.11022302462516E-16" rpy="0 0 0" />
+      <origin xyz="-0.0175869916443205 0 0" rpy="0 0 0" />
       <mass value="0.0194093358554489" />
       <inertia
@@ -191,5 +190,5 @@
     <parent link="right_truck_Link" />
     <child link="right_passive_sprocket_Link" />
-    <axis xyz="-1 0 0" />
+    <axis xyz="${reflect} 0 0" />
     <mimic joint="right_active_sprocket" multiplier="1" offset="0"/>
   </joint>
@@ -248,5 +247,5 @@
   </link>
   <joint name="right_truck_chain" type="fixed">
-    <origin xyz="0 0 0" rpy="0 0 3.54047866265369E-52" />
+    <origin xyz="0 0 0" rpy="0 0 0" />
     <parent link="right_truck_Link" />
     <child link="right_truck_chain_Link" />
