Commit message: Added Transmission for ros_control

File: ros_arvi_description/urdf/left_truck.urdf.xacro (robot description, xacro)
@@ -178,4 +178,24 @@
   </joint>
 </xacro:unless>
+		<transmission name="left_active_sprocket_trans" type="SimpleTransmission">
+			<type>transmission_interface/SimpleTransmission</type>
+			<actuator name="left_active_sprocket_motor">
+				<hardwareInterface>EffortJointInterface</hardwareInterface>
+				<mechanicalReduction>1</mechanicalReduction>
+			</actuator>
+			<joint name="left_active_sprocket">
+				<hardwareInterface>EffortJointInterface</hardwareInterface>
+			</joint>
+		</transmission>
+		<transmission name="left_passive_sprocket_trans" type="SimpleTransmission">
+			<type>transmission_interface/SimpleTransmission</type>
+			<actuator name="left_passive_sprocket_motor">
+				<hardwareInterface>EffortJointInterface</hardwareInterface>
+				<mechanicalReduction>1</mechanicalReduction>
+			</actuator>
+			<joint name="left_passive_sprocket">
+				<hardwareInterface>EffortJointInterface</hardwareInterface>
+			</joint>
+		</transmission>
   <link name="left_struct_truck_Link">
     <inertial>

File: ros_arvi_description/urdf/right_truck.urdf.xacro (robot description, xacro)
@@ -194,4 +194,24 @@
   </joint>
 </xacro:unless>
+		<transmission name="right_active_sprocket_trans" type="SimpleTransmission">
+			<type>transmission_interface/SimpleTransmission</type>
+			<actuator name="right_active_sprocket_motor">
+				<hardwareInterface>VelocityJointInterface</hardwareInterface>
+				<mechanicalReduction>1</mechanicalReduction>
+			</actuator>
+			<joint name="right_active_sprocket">
+				<hardwareInterface>VelocityJointInterface</hardwareInterface>
+			</joint>
+		</transmission>
+		<transmission name="right_passive_sprocket_trans" type="SimpleTransmission">
+			<type>transmission_interface/SimpleTransmission</type>
+			<actuator name="right_passive_sprocket_motor">
+				<hardwareInterface>VelocityJointInterface</hardwareInterface>
+				<mechanicalReduction>1</mechanicalReduction>
+			</actuator>
+			<joint name="right_passive_sprocket">
+				<hardwareInterface>VelocityJointInterface</hardwareInterface>
+			</joint>
+		</transmission>
   <link name="right_struct_truck_Link">
     <inertial>
