Commit message: Fixed name in urdf

File: arvi_description/urdf/arvi.urdf.xacro (robot description, xacro)
@@ -2,10 +2,10 @@
 <robot name="arvi_robot" xmlns:xacro="http://ros.org/wiki/xacro">
   <!-- Included URDF/XACRO Files -->
-  <xacro:include filename="$(find ros_arvi_description)/urdf/materials.urdf" />
-  <xacro:include filename="$(find ros_arvi_description)/urdf/left_truck.urdf.xacro" />
-  <xacro:include filename="$(find ros_arvi_description)/urdf/right_truck.urdf.xacro" />
-  <xacro:include filename="$(find ros_arvi_description)/urdf/plate.urdf.xacro" />
-  <xacro:include filename="$(find ros_arvi_description)/urdf/blades.urdf.xacro" />
-  <xacro:include filename="$(find ros_arvi_description)/urdf/tilt.urdf.xacro" />
+  <xacro:include filename="$(find arvi_description)/urdf/materials.urdf" />
+  <xacro:include filename="$(find arvi_description)/urdf/left_truck.urdf.xacro" />
+  <xacro:include filename="$(find arvi_description)/urdf/right_truck.urdf.xacro" />
+  <xacro:include filename="$(find arvi_description)/urdf/plate.urdf.xacro" />
+  <xacro:include filename="$(find arvi_description)/urdf/blades.urdf.xacro" />
+  <xacro:include filename="$(find arvi_description)/urdf/tilt.urdf.xacro" />
   <!-- Included URDF/XACRO Files -->
   <!-- Global properties -->
@@ -25,5 +25,5 @@
       <origin xyz="0 0 0" rpy="0 0 0" />
       <geometry>
-        <mesh filename="package://ros_arvi_description/meshes/body/base_link.STL" />
+        <mesh filename="package://arvi_description/meshes/body/base_link.STL" />
       </geometry>
       <material name="Yellow" />
@@ -32,5 +32,5 @@
       <origin xyz="0 0 0" rpy="0 0 0" />
       <geometry>
-        <mesh filename="package://ros_arvi_description/meshes/body/base_link.STL" />
+        <mesh filename="package://arvi_description/meshes/body/base_link.STL" />
       </geometry>
     </collision>
@@ -63,5 +63,5 @@
       <origin xyz="0 0 0" rpy="0 0 0" />
       <geometry>
-        <mesh filename="package://ros_arvi_description/meshes/body/body_part_Link.STL" />
+        <mesh filename="package://arvi_description/meshes/body/body_part_Link.STL" />
       </geometry>
       <material name="DarkGrey" />
@@ -70,5 +70,5 @@
       <origin xyz="0 0 0" rpy="0 0 0" />
       <geometry>
-        <mesh filename="package://ros_arvi_description/meshes/body/body_part_Link.STL" />
+        <mesh filename="package://arvi_description/meshes/body/body_part_Link.STL" />
       </geometry>
     </collision>
@@ -95,5 +95,5 @@
       <origin xyz="0 0 0" rpy="0 0 0" />
       <geometry>
-        <mesh filename="package://ros_arvi_description/meshes/body/electronics_body_Link.STL" />
+        <mesh filename="package://arvi_description/meshes/body/electronics_body_Link.STL" />
       </geometry>
       <material name="Green" />
@@ -102,5 +102,5 @@
       <origin xyz="0 0 0" rpy="0 0 0" />
       <geometry>
-        <mesh filename="package://ros_arvi_description/meshes/body/electronics_body_Link.STL" />
+        <mesh filename="package://arvi_description/meshes/body/electronics_body_Link.STL" />
       </geometry>
     </collision>
@@ -127,5 +127,5 @@
       <origin xyz="0 0 0" rpy="0 0 0" />
       <geometry>
-        <mesh filename="package://ros_arvi_description/meshes/body/black_body_Link.STL" />
+        <mesh filename="package://arvi_description/meshes/body/black_body_Link.STL" />
       </geometry>
       <material name="Black" />
@@ -134,5 +134,5 @@
       <origin xyz="0 0 0" rpy="0 0 0" />
       <geometry>
-        <mesh filename="package://ros_arvi_description/meshes/body/black_body_Link.STL" />
+        <mesh filename="package://arvi_description/meshes/body/black_body_Link.STL" />
       </geometry>
     </collision>
@@ -159,5 +159,5 @@
       <origin xyz="0 0 0" rpy="0 0 0" />
       <geometry>
-        <mesh filename="package://ros_arvi_description/meshes/body/cover_Link.STL" />
+        <mesh filename="package://arvi_description/meshes/body/cover_Link.STL" />
       </geometry>
       <material name="">
@@ -168,5 +168,5 @@
       <origin xyz="0 0 0" rpy="0 0 0" />
       <geometry>
-        <mesh filename="package://ros_arvi_description/meshes/body/cover_Link.STL" />
+        <mesh filename="package://arvi_description/meshes/body/cover_Link.STL" />
       </geometry>
     </collision>
@@ -196,5 +196,5 @@
       <origin xyz="0 0 0" rpy="0 0 0" />
       <geometry>
-        <mesh filename="package://ros_arvi_description/meshes/body/base_camera_Link.STL" />
+        <mesh filename="package://arvi_description/meshes/body/base_camera_Link.STL" />
       </geometry>
       <material name="Black" />
@@ -203,5 +203,5 @@
       <origin xyz="0 0 0" rpy="0 0 0" />
       <geometry>
-        <mesh filename="package://ros_arvi_description/meshes/body/base_camera_Link.STL" />
+        <mesh filename="package://arvi_description/meshes/body/base_camera_Link.STL" />
       </geometry>
     </collision>

File: arvi_description/urdf/blades.urdf.xacro (robot description, xacro)
@@ -1,5 +1,5 @@
 <?xml version="1.0"?>
 <robot xmlns:xacro="http://ros.org/wiki/xacro" name="blades">
-  <xacro:property name="path_blades" value="package://ros_arvi_description/meshes/blades" />
+  <xacro:property name="path_blades" value="package://arvi_description/meshes/blades" />
   <xacro:macro name="blades" params="parent">
   <link

File: arvi_description/urdf/description.xacro (robot description, xacro)
@@ -25,5 +25,5 @@
   <xacro:arg name="plate_enabled" default="true" />
   <xacro:arg name="truck_fixed" default="false" />
-  <xacro:include filename="$(find ros_arvi_description)/urdf/arvi.urdf.xacro" />
+  <xacro:include filename="$(find arvi_description)/urdf/arvi.urdf.xacro" />
   <xacro:arvi_robot />
 </robot>

File: arvi_description/urdf/left_truck.urdf.xacro (robot description, xacro)
@@ -1,5 +1,5 @@
 <?xml version="1.0"?>
 <robot xmlns:xacro="http://ros.org/wiki/xacro" name="left_truck">
-  <xacro:property name="path_left_truck" value="package://ros_arvi_description/meshes/left_truck" />
+  <xacro:property name="path_left_truck" value="package://arvi_description/meshes/left_truck" />
   <xacro:macro name="left_truck" params="parent reflect wheel_off *joint_pose">
   <link

File: arvi_description/urdf/plate.urdf.xacro (robot description, xacro)
@@ -1,5 +1,5 @@
 <?xml version="1.0"?>
 <robot xmlns:xacro="http://ros.org/wiki/xacro" name="plate">
-  <xacro:property name="path_plate" value="package://ros_arvi_description/meshes/plate" />
+  <xacro:property name="path_plate" value="package://arvi_description/meshes/plate" />
   <xacro:macro name="plate" params="parent">
   <link

File: arvi_description/urdf/right_truck.urdf.xacro (robot description, xacro)
@@ -1,5 +1,5 @@
 <?xml version="1.0"?>
 <robot xmlns:xacro="http://ros.org/wiki/xacro" name="right_truck">
-  <xacro:property name="path_right_truck" value="package://ros_arvi_description/meshes/right_truck" />
+  <xacro:property name="path_right_truck" value="package://arvi_description/meshes/right_truck" />
   <xacro:macro name="right_truck" params="parent reflect wheel_off *joint_pose">
   <link name="right_truck_Link">

File: arvi_description/urdf/tilt.urdf.xacro (robot description, xacro)
@@ -1,5 +1,5 @@
 <?xml version="1.0"?>
 <robot xmlns:xacro="http://ros.org/wiki/xacro" name="tilt">
-  <xacro:property name="path_tilt" value="package://ros_arvi_description/meshes/tilt" />
+  <xacro:property name="path_tilt" value="package://arvi_description/meshes/tilt" />
   <xacro:macro name="tilt" params="parent">
   <link

File: arvi_description/urdf/truck.urdf.xacro (robot description, xacro)
@@ -6,5 +6,5 @@
         <origin xyz="0 0 0" rpy="0 0 0" />
           <geometry>
-            <mesh filename="package://ros_arvi_description/meshes/truck/${position}_truck_link.STL" />
+            <mesh filename="package://arvi_description/meshes/truck/${position}_truck_link.STL" />
           </geometry>
           <material name="Yellow" />
@@ -13,5 +13,5 @@
         <origin xyz="0 0 0" rpy="0 0 0" />
         <geometry>
-          <mesh filename="package://ros_arvi_description/meshes/truck/${position}_truck_link.STL" />
+          <mesh filename="package://arvi_description/meshes/truck/${position}_truck_link.STL" />
         </geometry>
       </collision>
@@ -59,5 +59,5 @@
       <origin xyz="0 0 0" rpy="0 0 0" />
       <geometry>
-        <mesh filename="package://ros_arvi_description/meshes/truck/${position}_sprocket_link.STL" />
+        <mesh filename="package://arvi_description/meshes/truck/${position}_sprocket_link.STL" />
       </geometry>
       <material name="Black" />
@@ -66,5 +66,5 @@
       <origin xyz="0 0 0" rpy="0 0 0" />
       <geometry>
-        <mesh filename="package://ros_arvi_description/meshes/truck/${position}_sprocket_link.STL" />
+        <mesh filename="package://arvi_description/meshes/truck/${position}_sprocket_link.STL" />
       </geometry>
     </collision>
@@ -91,5 +91,5 @@
       <origin xyz="0 0 0" rpy="0 0 0" />
       <geometry>
-        <mesh filename="package://ros_arvi_description/meshes/truck/${position}_struct_truck_link.STL" />
+        <mesh filename="package://arvi_description/meshes/truck/${position}_struct_truck_link.STL" />
       </geometry>
       <material name="DarkGrey" />
@@ -98,5 +98,5 @@
       <origin xyz="0 0 0" rpy="0 0 0" />
       <geometry>
-        <mesh filename="package://ros_arvi_description/meshes/truck/${position}_struct_truck_link.STL" />
+        <mesh filename="package://arvi_description/meshes/truck/${position}_struct_truck_link.STL" />
       </geometry>
     </collision>
@@ -123,5 +123,5 @@
       <origin xyz="0 0 0" rpy="0 0 0" />
       <geometry>
-        <mesh filename="package://ros_arvi_description/meshes/truck/${position}_truck_chain_link.STL" />
+        <mesh filename="package://arvi_description/meshes/truck/${position}_truck_chain_link.STL" />
       </geometry>
       <material name="Black" />
@@ -130,5 +130,5 @@
       <origin xyz="0 0 0" rpy="0 0 0" />
       <geometry>
-        <mesh filename="package://ros_arvi_description/meshes/truck/${position}_truck_chain_link.STL" />
+        <mesh filename="package://arvi_description/meshes/truck/${position}_truck_chain_link.STL" />
       </geometry>
     </collision>

Commit message: Added option to fix tilt camera

File: arvi_description/urdf/arvi.urdf.xacro (robot description, xacro)
@@ -20,4 +20,12 @@
   <property name="truck_offset_z" value="0.024"/>
   <!-- Wheels params -->
+  <!-- front camera params -->
+  <xacro:if value="$(arg truck_fixed)">
+    <property name="camera_axis" value="fixed"/>
+  </xacro:if>
+  <xacro:unless value="$(arg truck_fixed)">
+    <property name="camera_axis" value="revolute"/>
+  </xacro:unless>
+  <!-- front camera params -->
   <!-- base_link -->
   <link name="base_link">
@@ -180,5 +188,5 @@
   <!-- Body chassis -->
   <!-- Cameras -->
-  <xacro:tilt parent="base_link"/>
+  <xacro:tilt parent="base_link" type="${camera_axis}"/>
   <link name="base_camera_Link">
     <inertial>

File: arvi_description/urdf/description.xacro (robot description, xacro)
@@ -25,4 +25,5 @@
   <xacro:arg name="plate_enabled" default="true" />
   <xacro:arg name="truck_fixed" default="false" />
+  <xacro:arg name="camera_fixed" default="false" />
   <xacro:include filename="$(find arvi_description)/urdf/arvi.urdf.xacro" />
   <xacro:arvi_robot />

File: arvi_description/urdf/tilt.urdf.xacro (robot description, xacro)
@@ -2,5 +2,5 @@
 <robot xmlns:xacro="http://ros.org/wiki/xacro" name="tilt">
   <xacro:property name="path_tilt" value="package://arvi_description/meshes/tilt" />
-  <xacro:macro name="tilt" params="parent">
+  <xacro:macro name="tilt" params="parent type">
   <link
     name="tilt_Link">
@@ -43,5 +43,5 @@
     </collision>
   </link>
-  <joint name="tilt" type="revolute">
+  <joint name="tilt" type="${type}">
     <origin xyz="0.227255888156922 0.016275 0.02745" rpy="1.5707963267949 3.80168975285532E-18 1.5707963267949" />
     <parent link="base_link" />
